File: hardware/NerdClock/_autosave-NerdClock.sch (KiCad schematic (older format))
At the start: 86 parts, among them J1 Conn_01x02, J10 Conn_01x04, J2 Jack-DC, J3 ICSP, J4 Conn_01x04, J5 Conn_01x03, J6 Conn_01x03, J7 USB_B_Micro, J8 Conn_01x02, J9 Conn_01x05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

Commit message: Added breakout tabs
Parts:
- added H10, H7, H8, H9: MountingHole, MountingHole:MountingHole_3.2mm_M3, symbol Mechanical:MountingHole
Changed lines of the file:
@@
 Wire Wire Line
 	9450 6200 9750 6200
+$Comp
+L Mechanical:MountingHole H9
+U 1 1 617FC01D
+P 8450 6050
+F 0 "H9" H 8550 6050 50  0000 L CNN
+F 1 "MountingHole" H 8550 6005 50  0001 L CNN
+F 2 "MountingHole:MountingHole_3.2mm_M3" H 8450 6050 50  0001 C CNN
+F 3 "~" H 8450 6050 50  0001 C CNN
+	1    8450 6050
+	1    0    0    -1
+$EndComp
+$Comp
+L Mechanical:MountingHole H10
+U 1 1 617FC375
+P 8800 6050
+F 0 "H10" H 8900 6050 50  0000 L CNN
+F 1 "MountingHole" H 8900 6005 50  0001 L CNN
+F 2 "MountingHole:MountingHole_3.2mm_M3" H 8800 6050 50  0001 C CNN
+F 3 "~" H 8800 6050 50  0001 C CNN
+	1    8800 6050
+	1    0    0    -1
+$EndComp
+$Comp
+L Mechanical:MountingHole H8
+U 1 1 6180746A
+P 8100 6050
+F 0 "H8" H 8200 6050 50  0000 L CNN
+F 1 "MountingHole" H 8200 6005 50  0001 L CNN
+F 2 "MountingHole:MountingHole_3.2mm_M3" H 8100 6050 50  0001 C CNN
+F 3 "~" H 8100 6050 50  0001 C CNN
+	1    8100 6050
+	1    0    0    -1
+$EndComp
+$Comp
+L Mechanical:MountingHole H7
+U 1 1 61807D5D
+P 7750 6050
+F 0 "H7" H 7850 6050 50  0000 L CNN
+F 1 "MountingHole" H 7850 6005 50  0001 L CNN
+F 2 "MountingHole:MountingHole_3.2mm_M3" H 7750 6050 50  0001 C CNN
+F 3 "~" H 7750 6050 50  0001 C CNN
+	1    7750 6050
+	1    0    0    -1
+$EndComp
 $EndSCHEMATC
