File: hardware/NerdClock/_autosave-NerdClock.sch (KiCad schematic (older format))
At the start: 95 parts, among them J1 Conn_01x02, J10 Conn_01x04, J11 Conn_01x02, J12 Conn_01x02, J2 Jack-DC, J3 ICSP, J4 Conn_01x04, J5 Conn_01x02, J6 Conn_01x02, J7 USB_B_Micro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

Commit message: Routing probably done?
Changed lines of the file:
@@
 $Comp
 L Graphic:Logo_Open_Hardware_Large #LOGO?
-U 1 1 620E6705
-P 10500 3900
-F 0 "#LOGO?" H 10500 4400 50  0001 C CNN
-F 1 "Logo_Open_Hardware_Large" H 10500 3500 50  0001 C CNN
-F 2 "" H 10500 3900 50  0001 C CNN
-F 3 "~" H 10500 3900 50  0001 C CNN
-	1    10500 3900
+U 1 1 6210449D
+P 10650 4100
+F 0 "#LOGO?" H 10650 4600 50  0001 C CNN
+F 1 "Logo_Open_Hardware_Large" H 10650 3700 50  0001 C CNN
+F 2 "" H 10650 4100 50  0001 C CNN
+F 3 "~" H 10650 4100 50  0001 C CNN
+	1    10650 4100
 	1    0    0    -1
 $EndComp
